File: hw/usb-rs485_switch/485_line_driver.sch (KiCad schematic (older format))
At the start: 21 parts

Commit message: Progress in schematic.
Parts:
- added C?: 100n, symbol Device:C
- added JP? (x2): SolderJumper_2_Open, symbol Jumper:SolderJumper_2_Open
- added R?: 10k, symbol Device:R
- added R?: 100k, symbol Device:R
- R? (x2): value R -> 720R
- R?: value R -> 120R
Connections:
- net +5V: now also JP?.1 (A)
- net GND: now also C?.2, JP?.2 (B), R?.2
- net I_SENSE: now also C?.1, R?.1
- net PWR_EN: now also R?.1
- net at F?.2, U?.6 (A): now also R?.1, R?.2
- net at F?.2, U?.7 (B): now also R?.1, R?.2
- net at R?.1: now also JP?.2 (B)
- net at R?.2: now also JP?.1 (A)
- net at U?.1: now also R?.2
