File: hw/usb-rs485_switch/usb-rs485_switch.sch (KiCad schematic (older format))
At the start: 20 parts

Commit message: Schematic WIP.
Parts:
- removed U?: 74HC138, symbol 74xx:74LS138
- added C? (x3): C, symbol Device:C
- added C? (x5): 100n, symbol Device:C
- added D?: VCC_LED, symbol Device:LED
- added D?: 5V_LED, symbol Device:LED
- added D?: 3V3_LED, symbol Device:LED
- added D?: USR_LED, symbol Device:LED
- added J? (x2): RJ45_LED_Shielded, symbol Connector:RJ45_LED_Shielded
- added JP?: SolderJumper_2_Open, symbol Jumper:SolderJumper_2_Open
- added R? (x8): 1k, symbol Device:R
- added R? (x8): R, symbol Device:R
- added U? (x3): 74HC595, symbol 74xx:74HC595
- added U?: CD4051B, symbol Analog_Switch:CD4051B
Connections:
- net +3V3: now also U?.10 (~SRCLR), U?.16 (VCC), C?.1, C?.1, C?.1, C?.1, C?.1, R?.1, R?.1, U?.10 (~SRCLR), U?.10 (~SRCLR), U?.10 (~SRCLR), U?.16 (VCC), U?.16 (VCC), U?.16 (VCC), U?.16 (VDD)
- net +5V: now also R?.1, R?.1
- net GND: now also U?.15 (GND2), U?.8 (GND), U?.9 (GND2), C?.2, C?.2, C?.2, C?.2, C?.2, C?.2, D?.1 (K), D?.1 (K), D?.1 (K), R?.2, R?.2, U?.6 (INH), U?.7 (VEE), U?.8 (GND), U?.8 (GND), U?.8 (GND), U?.8 (VSS)
- net GND2: now also U?.2 (GND1), U?.8 (GND1), C?.2, C?.2
- net VCC_SENSE: now reaches U?.10 (PA0)
- net VCC_SENSE: now also R?.1, R?.2
- net 5V_SENSE: now reaches U?.11 (PA1)
- net 5V_SENSE: now also R?.1, R?.2
- net USART2_TX: now reaches U?.12 (PA2)
- net USART2_RX: now reaches U?.13 (PA3)
- net AIN8: now reaches U?.18 (PB0)
- net I_SENSE: now reaches U?.19 (PB1)
- net I_SENSE: now also U?.3 (X)
- net at U?.2 (PC13): now also D?.1 (K)
- net BOOT1: now reaches U?.20 (PB2)
- net USART3_TX: now reaches U?.21 (PB10)
- net USART3_RX: now reaches U?.22 (PB11)
- net SPI2_STROBE: now reaches U?.25 (PB12)
- net SPI2_STROBE: now also U?.12 (RCLK), U?.12 (RCLK), U?.12 (RCLK), U?.12 (RCLK)
- net SPI2_SCK: now reaches U?.26 (PB13)
- net SPI2_SCK: now also U?.11 (SRCLK), U?.11 (SRCLK), U?.11 (SRCLK), U?.11 (SRCLK)
- net SPI2_MISO: now reaches U?.27 (PB14)
- net SPI2_MOSI: now reaches U?.28 (PB15)
- net SPI2_MOSI: now also U?.14 (SER)
- net ~SPI2_OE: now reaches U?.29 (PA8)
- net ~SPI2_OE: now also U?.13 (~OE), U?.13 (~OE), U?.13 (~OE), U?.13 (~OE)
- net USART1_TX: now reaches U?.30 (PA9)
- net USART1_RX: now reaches U?.31 (PA10)
- net USB_DN: now reaches U?.32 (PA11)
- net USB_DN: now also R?.1
- net USB_DP: now reaches U?.33 (PA12)
- net USB_DP: now also R?.1
- net SWDIO: now reaches U?.34 (PA13)
- net SWCLK: now reaches U?.37 (PA14)
- net I_SEN_A: now reaches U?.39 (PB3)
- net I_SEN_A: now also U?.11 (A)
- net I_SEN_B: now reaches U?.40 (PB4)
- net I_SEN_B: now also U?.10 (B)
- net I_SEN_C: now reaches U?.41 (PB5)
- net I_SEN_C: now also U?.9 (C)
- net I2C1_SCL: now reaches U?.42 (PB6)
- net I2C1_SDA: now reaches U?.43 (PB7)
- net at U?.1 (VBUS1): now also C?.1
- net at U?.10 (DD+): now also R?.2
- net at U?.11 (DD-): now also R?.2
- net at U?.13 (SPD): now also U?.14 (VDD2), C?.1
- net at U?.3 (VDD1): now also U?.4 (PDEN), U?.5 (SPU), C?.1
- net at U?.6 (UD-): now also R?.1
- net at U?.7 (UD+): now also R?.1
- net at U?.1 (QB): now also R?.2
- net at U?.15 (QA): now also R?.2
- net at U?.2 (QC): now also R?.2
- net at U?.3 (QD): now also R?.2
- net at U?.4 (QE): now also R?.2
- net at U?.5 (QF): now also R?.2
- net at U?.6 (QG): now also R?.2
- net at U?.7 (QH): now also R?.2
- net at U?.9 (QH'): now also U?.14 (SER)
- new net: U?.14 (SER), U?.9 (QH') (x2)
- new net: D?.2 (A), R?.2 (x4)
- new net I_SENSE1: U?.13 (X0)
- new net I_SENSE2: U?.14 (X1)
- new net I_SENSE3: U?.15 (X2)
- new net I_SENSE4: U?.12 (X3)
- new net I_SENSE5: U?.1 (X4)
- new net I_SENSE6: U?.5 (X5)
- new net I_SENSE7: U?.2 (X6)
- new net I_SENSE8: U?.4 (X7)
- new net LED_G1: R?.1
- new net LED_G2: R?.1
- new net LED_G3: R?.1
- new net LED_G4: R?.1
- new net LED_G5: R?.1
- new net LED_G6: R?.1
- new net LED_G7: R?.1
- new net LED_G8: R?.1
- new net PWR_EN1: U?.15 (QA)
- new net PWR_EN2: U?.1 (QB)
- new net PWR_EN3: U?.2 (QC)
- new net PWR_EN4: U?.3 (QD)
- new net PWR_EN5: U?.4 (QE)
- new net PWR_EN6: U?.5 (QF)
- new net PWR_EN7: U?.6 (QG)
- new net PWR_EN8: U?.7 (QH)
- new net TX_EN1: U?.15 (QA)
- new net TX_EN2: U?.1 (QB)
- new net TX_EN3: U?.2 (QC)
- new net TX_EN4: U?.3 (QD)
- new net TX_EN5: U?.4 (QE)
- new net TX_EN6: U?.5 (QF)
- new net TX_EN7: U?.6 (QG)
- new net TX_EN8: U?.7 (QH)
- new net VCC: R?.1, R?.1
- new net ~RX_EN1: U?.15 (QA)
- new net ~RX_EN2: U?.1 (QB)
- new net ~RX_EN3: U?.2 (QC)
- new net ~RX_EN4: U?.3 (QD)
- new net ~RX_EN5: U?.4 (QE)
- new net ~RX_EN6: U?.5 (QF)
- new net ~RX_EN7: U?.6 (QG)
- new net ~RX_EN8: U?.7 (QH)
Other:
- note added: "K MCU"
- note added: "K pocitaci"
- moved on the sheet: R?, U?

Commit message: Progress in schematic.
Parts:
- added C?: 180u, symbol Device:CP
- added C?: 1u, symbol Device:C
- added C?: 470u, symbol Device:CP
- added C?: CP, symbol Device:CP
- added C?: 10n, symbol Device:C
- added C?: 220u, symbol Device:CP
- added D? (x2): D_Schottky, symbol Device:D_Schottky
- added D?: SM6T27A, Diode_SMD:D_SMB, symbol Diode:SM6T27A
- added D?: 40V/3A, symbol Device:D_Schottky
- added F?: Polyfuse, symbol Device:Polyfuse
- added J?: POWER, symbol Connector:Conn_01x02_Male
- added J?: PROG, symbol Connector:Conn_01x05_Male
- added J?: USART2, symbol Connector:Conn_01x05_Male
- added J?: I2C, symbol Connector:Conn_01x04_Male
- added J?: VCC_OUT1, symbol Connector:Conn_01x02_Male
- added J?: VCC_OUT2, symbol Connector:Conn_01x02_Male
- added J?: 5V_OUT1, symbol Connector:Conn_01x02_Male
- added J?: 5V_OUT2, symbol Connector:Conn_01x02_Male
- added J?: 3V_OUT1, symbol Connector:Conn_01x02_Male
- added J?: 3V3_OUT2, symbol Connector:Conn_01x02_Male
- added J?: SPI, symbol Connector:Conn_01x06_Male
- added J?: GPIO, symbol Connector:Conn_01x06_Male
- added L?: 68u/3A, symbol Device:L
- added L?: 22u, symbol Device:L
- added R? (x7): R, symbol Device:R
- added R? (x2): 4k7, symbol Device:R
- added R? (x9): 330R, symbol Device:R
- added TP?: NRST, symbol Connector:TestPoint
- added TP?: BOOT0, symbol Connector:TestPoint
- added U?: XL1509-5.0E1, Package_SO:SO-8_5.3x6.2mm_P1.27mm, symbol xl1509:XL1509-5.0E1
- added U?: TPS5430DDA, Package_SO:TI_SO-PowerPAD-8_ThermalVias, symbol Regulator_Switching:TPS5430DDA
- added U?: M24C01-WMN, Package_SO:SOIC-8_3.9x4.9mm_P1.27mm, symbol Memory_EEPROM:M24C01-WMN
Connections:
- net +3V3: now also J?.1 (Pin_1), J?.1 (Pin_1), J?.4 (Pin_4), J?.4 (Pin_4), J?.5 (Pin_5), J?.6 (Pin_6), J?.6 (Pin_6), R?.1, R?.1, U?.8 (VCC)
- net +5V: now also C?.1, C?.1, J?.1 (Pin_1), J?.1 (Pin_1), J?.4 (Pin_4), L?.2, L?.2, R?.1, U?.3 (FB)
- net GND: now also C?.2, C?.2, C?.2, C?.2, C?.2, D?.2 (A), D?.2 (A), D?.2 (A2), J?.1 (Pin_1), J?.2 (Pin_2), J?.2 (Pin_2), J?.2 (Pin_2), J?.2 (Pin_2), J?.2 (Pin_2), J?.2 (Pin_2), J?.2 (Pin_2), J?.3 (Pin_3), J?.3 (Pin_3), J?.5 (Pin_5), J?.5 (Pin_5), R?.2, R?.2, R?.2, R?.2, U?.1 (E0), U?.2 (E1), U?.3 (E2), U?.4 (On/Off), U?.4 (VSS), U?.5 (GND), U?.6 (GND), U?.6 (GND), U?.7 (GND), U?.8 (GND), U?.9 (GNDPAD)
- net I2C1_SCL: now also J?.2 (Pin_2), R?.2, U?.6 (SCL)
- net I2C1_SDA: now also J?.1 (Pin_1), R?.2, U?.5 (SDA)
- net SWCLK: now also J?.2 (Pin_2), R?.1; no longer U?.37 (PA14)
- net SWDIO: now also J?.3 (Pin_3), R?.1; no longer U?.34 (PA13)
- net USART2_RX: now also R?.1, R?.1; no longer U?.13 (PA3)
- net USART2_TX: now also R?.1, R?.1; no longer U?.12 (PA2)
- net VCC: now also C?.1, C?.1, C?.1, D?.1 (K), J?.1 (Pin_1), J?.1 (Pin_1), U?.1 (Input), U?.7 (VIN)
- net at U?.14 (PA4): now also R?.2
- net at U?.15 (PA5): now also R?.2
- net at U?.16 (PA6): now also R?.2
- net at U?.17 (PA7): now also R?.2
- net at U?.38 (PA15): now also R?.2
- net at U?.44 (BOOT0): now also R?.1, TP?.1
- net GPIO1: now reaches U?.45 (PB8)
- net GPIO1: now also J?.2 (Pin_2)
- net GPIO2: now reaches U?.46 (PB9)
- net GPIO2: now also J?.3 (Pin_3)
- net NRST: now reaches R?.2, U?.7 (NRST)
- net NRST: now also J?.5 (Pin_5), TP?.1
- net AIN8 renamed GPIO0
- net GPIO0: now also J?.1 (Pin_1)
- new net: R?.2, U?.12 (PA2)
- new net: R?.2, U?.13 (PA3)
- new net: R?.2, U?.34 (PA13)
- new net: R?.2, U?.37 (PA14)
- new net: D?.1 (K), L?.1, U?.2 (Output)
- new net: D?.1 (A1), F?.2, J?.1 (Pin_1)
- new net: D?.2 (A), F?.1
- new net: J?.1 (Pin_1), R?.1, R?.2
- new net: J?.2 (Pin_2), R?.2
- new net: C?.1, U?.1 (BOOT)
- new net: R?.1, R?.2, U?.4 (VSENSE)
- new net: C?.2, D?.1 (K), L?.1, U?.8 (PH)
- new net: R?.1, U?.7 (~WC)
- new net GPIO3: J?.4 (Pin_4), R?.1
- new net SPI1_MISO: J?.3 (Pin_3), R?.1
- new net SPI1_MOSI: J?.4 (Pin_4), R?.1
- new net SPI1_SCK: J?.2 (Pin_2), R?.1
- new net ~SPI1_SS: J?.1 (Pin_1), R?.1
Other:
- note added: "1.221V"
- note added: "TODO: USB"
- moved on the sheet: C?, D?, JP?, R?, U?
