File: hw/usb-rs485_switch/usb-rs485_switch.kicad_pcb (KiCad board)
At the start: 2 copper layers, 347 parts, among them J1 RJ45_LED_Shielded, J10 VCC_OUT2, J11 5V_OUT1, J12 5V_OUT2, J13 3V_OUT1, J14 3V3_OUT2, J15 MC-107DM, J16 RES1, J17 USB_NONISO, J18 RJ45_LED_Shielded, J19 RJ45_LED_Shielded, J2 RJ45_LED_Shielded, J20 RJ45_LED_Shielded, J21 RJ45_LED_Shielded, J22 RJ45_LED_Shielded, J23 RJ45_LED_Shielded, J24 1WIRE_CHANNELS, J25 USB_ISO, J26 RES2, J27 USART3, J28 RES3, J29 RES4, J3 USART2, J30 RES5, J31 RES6, J32 RES7, J33 RES8, J34 1WIRE_SELECT, J35 USB-C_SBU, J36 PWR_SELECT, J4 I2C, J5 SPI, J6 GPIO, J7 PROG, J8 POWER, J9 VCC_OUT1, Q1 MMBT5551, Q10 Si2301CDS, Q11 MMBT5551, Q12 Si2301CDS, Q13 MMBT5551, Q14 Si2301CDS, Q15 MMBT5551, Q16 Si2301CDS, Q2 Si2301CDS, Q3 MMBT5551, Q4 Si2301CDS, Q5 MMBT5551, Q6 Si2301CDS, Q7 MMBT5551, Q8 Si2301CDS, Q9 MMBT5551, U1 74HC595, U10 XL1509-5.0E1, U11 AMS1117-3.3, U12 INA180A1, U13 MAX485E, U14 INA180A1, U15 MAX485E, U16 INA180A1, U17 MAX485E, U18 INA180A1, U19 MAX485E, U2 CD4051B, U20 INA180A1, U21 MAX485E, U22 INA180A1, U23 MAX485E, U24 INA180A1, U25 MAX485E, U26 INA180A1, U27 MAX485E, U28 SRV05-4, U29 SRV05-4, U3 74HC595, U4 74HC595, U5 74HC595, U6 STM32F103C8Tx, U7 ADUM4160, U8 M24C01-WMN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

Commit message: Routing in progress.
Parts:
- added C1: 100n, Capacitor_SMD:C_0603_1608Metric, F.Cu at (144.5, 45.5)
- added C2: 100n, Capacitor_SMD:C_0603_1608Metric, F.Cu at (210.8, 73.2)
- added C3: 100n, Capacitor_SMD:C_0603_1608Metric, F.Cu at (180.3, 46.0)
- added H1: MountingHole_Pad, MountingHole:MountingHole_3.2mm_M3_Pad_Via, F.Cu at (125.0, 15.0)
- added H2: MountingHole_Pad, MountingHole:MountingHole_3.2mm_M3_Pad_Via, F.Cu at (290.0, 15.0)
- added H3: MountingHole_Pad, MountingHole:MountingHole_3.2mm_M3_Pad_Via, F.Cu at (290.0, 65.0)
- added H4: MountingHole_Pad, MountingHole:MountingHole_3.2mm_M3_Pad_Via, F.Cu at (125.0, 65.0)
- moved J24 252.6 mm to (288.8, 21.8)
- moved J34 239.0 mm to (291.3, 43.4)
- moved PS1 223.5 mm to (253.0, 127.5), turned to 90 degrees
- moved J22 208.4 mm to (251.7, 16.1)
- moved J17 207.3 mm to (271.5, 107.9)
- moved R8 198.2 mm to (277.6, 26.6), turned to -90 degrees
- moved U29 197.2 mm to (280.3, 112.3)
- moved J23 187.4 mm to (271.4, 16.1)
- moved U5 184.8 mm to (265.0, 48.0), turned to -90 degrees
- moved U26 180.5 mm to (283.0, 33.4), turned to -90 degrees
- moved F23 176.6 mm to (280.8, 28.0), turned to 90 degrees
- moved R143 174.3 mm to (256.4, 26.6), turned to -90 degrees
- moved C24 173.8 mm to (215.1, 79.2), turned to 180 degrees
- moved R29 169.2 mm to (267.0, 109.2)
- moved F24 169.0 mm to (270.3, 30.6), turned to -90 degrees
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Connections:
- J24 pad 1: /1WIRE1 -> /1WIRE8
- J24 pad 11: /1WIRE6 -> /1WIRE3
- J24 pad 13: /1WIRE7 -> /1WIRE2
- J24 pad 15: /1WIRE8 -> /1WIRE1
- J24 pad 3: /1WIRE2 -> /1WIRE7
- J24 pad 5: /1WIRE3 -> /1WIRE6
- J24 pad 7: /1WIRE4 -> /1WIRE5
- J24 pad 9: /1WIRE5 -> /1WIRE4
- R1 pad 2: Net-(R1-Pad2) -> Net-(U1-Pad4)
- R2 pad 1: /LED_G2 -> /LED_G3
- R2 pad 2: Net-(R2-Pad2) -> Net-(U3-Pad4)
- R3 pad 1: /LED_G3 -> /LED_G4
- R3 pad 2: Net-(R3-Pad2) -> Net-(U3-Pad15)
- R4 pad 1: /LED_G4 -> /LED_G6
- R4 pad 2: Net-(R4-Pad2) -> Net-(U4-Pad15)
- R5 pad 1: /LED_G5 -> /LED_G2
- R5 pad 2: Net-(R5-Pad2) -> Net-(U1-Pad15)
- R6 pad 1: /LED_G6 -> /LED_G5
- R6 pad 2: Net-(R6-Pad2) -> Net-(U4-Pad4)
- U1 pad 1: Net-(R2-Pad2) -> /PWR_EN2
- U1 pad 15: Net-(R1-Pad2) -> Net-(U1-Pad15)
- U1 pad 2: Net-(R3-Pad2) -> /TX_EN2
- U1 pad 3: Net-(R4-Pad2) -> /~{RX_EN2}
- U1 pad 4: Net-(R5-Pad2) -> Net-(U1-Pad4)
- U1 pad 5: Net-(R6-Pad2) -> /PWR_EN1
- U1 pad 6: Net-(R7-Pad2) -> /TX_EN1
- U1 pad 7: Net-(R8-Pad2) -> /~{RX_EN1}
- U3 pad 1: /PWR_EN2 -> /PWR_EN4
- U3 pad 15: /PWR_EN1 -> Net-(U3-Pad15)
- U3 pad 2: /PWR_EN3 -> /TX_EN4
- U3 pad 3: /PWR_EN4 -> /~{RX_EN4}
- U3 pad 4: /PWR_EN5 -> Net-(U3-Pad4)
- U3 pad 5: /PWR_EN6 -> /PWR_EN3
- U3 pad 6: /PWR_EN7 -> /TX_EN3
- U3 pad 7: /PWR_EN8 -> /~{RX_EN3}
- U4 pad 1: /TX_EN2 -> /PWR_EN6
- U4 pad 15: /TX_EN1 -> Net-(U4-Pad15)
- U4 pad 2: /TX_EN3 -> /TX_EN6
- U4 pad 3: /TX_EN4 -> /~{RX_EN6}
- U4 pad 4: /TX_EN5 -> Net-(U4-Pad4)
- U4 pad 5: /TX_EN6 -> /PWR_EN5
- U4 pad 6: /TX_EN7 -> /TX_EN5
- U4 pad 7: /TX_EN8 -> /~{RX_EN5}
- U5 pad 1: /~{RX_EN2} -> /PWR_EN8
- U5 pad 15: /~{RX_EN1} -> Net-(R8-Pad2)
- U5 pad 2: /~{RX_EN3} -> /TX_EN8
- U5 pad 3: /~{RX_EN4} -> /~{RX_EN8}
- U5 pad 4: /~{RX_EN5} -> Net-(R7-Pad2)
- U5 pad 5: /~{RX_EN6} -> /PWR_EN7
- U5 pad 6: /~{RX_EN7} -> /TX_EN7
- U5 pad 7: /~{RX_EN8} -> /~{RX_EN7}
Routing:
- net /1WIRE3: track 0.00 -> 124.6 mm
- net /1WIRE4: track 0.00 -> 103.3 mm
- net /1WIRE5: track 0.00 -> 81.7 mm
- net /1WIRE6: track 0.00 -> 59.3 mm
- net /1WIRE7: track 0.00 -> 37.1 mm
- net /sheet62070CF7/A: track 0.00 -> 30.6 mm, vias 0 -> 1
- net /RS485 Line driver/A: track 0.00 -> 30.3 mm, vias 0 -> 1
- net /sheet6205AD21/A: track 0.00 -> 30.2 mm, vias 0 -> 1
- net /sheet620CBEF2/A: track 0.00 -> 30.2 mm, vias 0 -> 1
- net /sheet620CBEF4/A: track 0.00 -> 29.3 mm, vias 0 -> 1
- net /sheet620CBEF1/A: track 0.00 -> 29.0 mm, vias 0 -> 1
- net /sheet620AF7C7/A: track 0.00 -> 28.7 mm, vias 0 -> 1
- net /sheet620CBEF3/A: track 0.00 -> 28.6 mm, vias 0 -> 1
- net Net-(J19-Pad3): track 0.00 -> 25.8 mm
- net Net-(J23-Pad3): track 0.00 -> 25.7 mm
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- added copper zone on B.Cu, net GND
- added copper zone on F.Cu, net GND
Other:
- board outline added: 175 x 60 mm

Commit message: Routing in progress...
Parts:
- removed C17: 10n, Capacitor_SMD:C_0603_1608Metric
- removed D8, D9: SS54, Diode_SMD:D_SMA
- removed R154, R20: 330R, Resistor_SMD:R_0603_1608Metric
- removed R34, R39, R40: R, Resistor_SMD:R_0603_1608Metric
- removed TP2: NRST, TestPoint:TestPoint_THTPad_D2.0mm_Drill1.0mm
- removed U10: XL1509-5.0E1, Package_SO:SO-8_5.3x6.2mm_P1.27mm
- removed U9: TPS5430DDA, Package_SO:TI_SO-PowerPAD-8_ThermalVias
- added C51: 100n, Capacitor_SMD:C_0603_1608Metric, F.Cu at (189.8, 98.2)
- added C52: 100n, Capacitor_SMD:C_0603_1608Metric, F.Cu at (109.7, 97.8)
- added C58: 4u7/50V, Capacitor_SMD:C_1206_3216Metric, F.Cu at (101.8, 94.8)
- added C59: 8.2n, Capacitor_SMD:C_0603_1608Metric, F.Cu at (110.8, 101.4)
- added C60: 22n, Capacitor_SMD:C_0603_1608Metric, F.Cu at (112.4, 101.4)
- added C61: 8.2n, Capacitor_SMD:C_0603_1608Metric, F.Cu at (101.5, 102.6)
- added C62: 22u/6.3V X5R, Capacitor_SMD:C_0603_1608Metric, F.Cu at (109.8, 91.9)
- added C63: 4u7/50V, Capacitor_SMD:C_1206_3216Metric, F.Cu at (101.8, 97.2)
- added D26: SS14, Diode_SMD:D_SMA, F.Cu at (107.8, 95.1)
- added L3: 47u, Inductor_SMD:L_Bourns_SRP7028A_7.3x6.6mm, F.Cu at (115.0, 94.9)
- added R156: R, Resistor_SMD:R_0603_1608Metric, F.Cu at (111.5, 103.7)
- added R157: R, Resistor_SMD:R_0603_1608Metric, F.Cu at (114.8, 103.7)
- added R158: R, Resistor_SMD:R_0603_1608Metric, F.Cu at (113.9, 101.4)
- added U30: TPS54331, Package_SO:SOIC-8_3.9x4.9mm_P1.27mm, F.Cu at (106.1, 101.4)
- moved J3 142.5 mm to (199.4, 91.6)
- moved R149 141.8 mm to (226.2, 81.5)
- moved R148 134.2 mm to (223.2, 81.5)
- moved C13 132.3 mm to (151.5, 89.7), turned to 90 degrees
- moved J27 131.0 mm to (223.6, 84.1), turned to 90 degrees
- moved R147 125.5 mm to (205.9, 98.9), turned to 90 degrees
- moved U29 123.6 mm to (158.3, 92.5)
- moved PS1 121.6 mm to (134.7, 99.7)
- moved R146 119.8 mm to (120.5, 100.1), turned to 90 degrees
- moved C46 119.5 mm to (135.3, 96.9)
- moved J17 118.7 mm to (154.4, 88.6)
- moved R28 117.9 mm to (150.6, 95.2), turned to 180 degrees
- moved R29 117.4 mm to (150.6, 93.7), turned to 180 degrees
- moved C9 117.3 mm to (134.5, 89.6), turned to 90 degrees
- moved U7 117.0 mm to (143.0, 91.9)
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Connections:
- net Net-(J15-PadA6) renamed /USB_IN_P
- net Net-(J15-PadA7) renamed /USB_IN_N
- J3 pad 2: Net-(J3-Pad2) -> /USART2_TX
- J3 pad 4: +5V -> unconnected-(J3-Pad4)
- U2 pad 1: /I_SENSE5 -> /I_SENSE1
- U2 pad 12: /I_SENSE4 -> /I_SENSE8
- U2 pad 13: /I_SENSE1 -> /I_SENSE7
- U2 pad 14: /I_SENSE2 -> /I_SENSE6
- U2 pad 15: /I_SENSE3 -> /I_SENSE5
- U2 pad 2: /I_SENSE7 -> /I_SENSE3
- U2 pad 4: /I_SENSE8 -> /I_SENSE4
- U2 pad 5: /I_SENSE6 -> /I_SENSE2
- U29 pad 4: /1WIRE -> unconnected-(U29-Pad4)
- U6 pad 13: Net-(R20-Pad2) -> /USART2_RX
- U6 pad 27: Net-(R154-Pad1) -> unconnected-(U6-Pad27)
Routing:
- net +3V3: track 5.35 -> 548.8 mm, vias 0 -> 23
- net +5V: track 21.1 -> 358.4 mm, vias 0 -> 10
- net VCC: track 4.27 -> 287.3 mm, vias 0 -> 8
- net GND: track 0.00 -> 278.3 mm, vias 0 -> 85
- net /1WIRE1: track 0.00 -> 178.0 mm, vias 0 -> 1
- net /1WIRE2: track 0.00 -> 155.0 mm, vias 0 -> 1
- net /~{SPI2_OE}: track 0.00 -> 140.8 mm, vias 0 -> 5
- net /SPI2_STROBE: track 0.00 -> 133.3 mm, vias 0 -> 5
- net /SPI2_SCK: track 0.00 -> 131.7 mm, vias 0 -> 5
- net /USART1_TX: track 0.00 -> 102.4 mm, vias 0 -> 5
- net /USART1_RX: track 0.00 -> 99.3 mm, vias 0 -> 5
- net /USART3_TX: track 0.00 -> 92.6 mm, vias 0 -> 6
- net /USART3_RX: track 0.00 -> 91.6 mm, vias 0 -> 4
- net /1WIRE: track 0.00 -> 88.6 mm, vias 0 -> 1
- net Net-(R97-Pad2): track 0.00 -> 78.2 mm, vias 0 -> 4
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- added copper zone on F.Cu, net +3V3
- added copper zone on B.Cu, net GND2
- added copper zone on F.Cu, net GND2
Other:
- outline, holes or cut-outs redrawn
