File: hw/usb-rs485_switch/usb-rs485_switch.kicad_sch (KiCad schematic)
At the start: 150 parts, among them J1 RJ45_LED_Shielded, J10 VCC_OUT2, J11 5V_OUT1, J12 5V_OUT2, J13 3V_OUT1, J14 3V3_OUT2, J15 MC-107DM, J16 RES1, J17 USB_NONISO, J18 RJ45_LED_Shielded, J19 RJ45_LED_Shielded, J2 RJ45_LED_Shielded, J20 RJ45_LED_Shielded, J21 RJ45_LED_Shielded, J22 RJ45_LED_Shielded, J23 RJ45_LED_Shielded, J24 1WIRE_CHANNELS, J25 USB_ISO, J26 RES2, J27 USART3, J28 RES3, J29 RES4, J3 USART2, J30 RES5, J31 RES6, J32 RES7, J33 RES8, J34 1WIRE_SELECT, J35 USB-C_SBU, J36 PWR_SELECT, J4 I2C, J5 SPI, J6 GPIO, J7 PROG, J8 POWER, J9 VCC_OUT1, U1 74HC595, U11 AMS1117-3.3, U2 CD4051B, U28 SRV05-4, U29 SRV05-4, U3 74HC595, U30 TPS54331, U4 74HC595, U5 74HC595, U6 STM32F103C8Tx, U7 ADUM4160, U8 M24C01-WMN, Y1 Crystal_GND23

Commit message: Final changes.
Parts:
- C1, C10, C11, C12, C13, C2, C3, C4, C48, C49, C5, C51, C52, C8, C9: LCSC (none) -> C14663
- C16, C47: LCSC (none) -> C19702
- C18: value CP -> 330u; footprint (none) -> Capacitor_THT:CP_Radial_D10.0mm_P5.00mm
- C19: LCSC (none) -> C59461
- C46, C63: LCSC (none) -> C29823
- C50: LCSC (none) -> C15849
- C59, C61: LCSC (none) -> C27920
- C6, C7: value C -> 20pF; LCSC (none) -> C1648
- C60: LCSC (none) -> C21122
- D2: LCSC (none) -> C133693
- F1: value Polyfuse -> SHV2920P500-30-AA; LCSC (none) -> C495350
- J18, J19, J2, J20, J21, J22, J23: LCSC (none) -> C386757
- R1, R2, R3, R4, R5, R6, R7, R8: LCSC (none) -> C21190
- R10, R11, R15, R157, R16, R35, R36, R9: value R -> 10k; LCSC (none) -> C25804
- R12, R13, R38: value R -> 1k; LCSC (none) -> C21190
- R137, R138, R139, R140, R141, R142, R143, R144: LCSC (none) -> C13167
- R14: value R -> 1M; LCSC (none) -> C22935
- R145, R146: LCSC (none) -> C23186
- R147, R30, R33: LCSC (none) -> C23162
- R148, R149: value R -> 330R; LCSC (none) -> C23138
- R150, R151, R152, R153, R19, R21, R22, R23, R24, R25, R26, R27: LCSC (none) -> C23138
- R156: value R -> 100R; LCSC (none) -> C22775
- R158: value R -> 1k8; LCSC (none) -> C4177
- R17, R18, R28, R29: LCSC (none) -> C23345
- R31, R37: value R -> 2k7; LCSC (none) -> C13167
- R32: value R -> 4k7; LCSC (none) -> C23162
- U11: LCSC (none) -> C6186
- U28, U29: LCSC (none) -> C85364
- U30: LCSC (none) -> C9865
